Commit message: Imported upstream version '0.8.2' of 'upstream'

File: franka_description/robots/dual_panda_example.urdf.xacro (robot description, xacro)
@@ -25,7 +25,7 @@
   <!-- right arm with gripper -->
   <xacro:panda_arm arm_id="$(arg arm_id_1)" connected_to="base"  xyz="0 -0.5 1" safety_distance="0.03"/>
-  <xacro:hand ns="$(arg arm_id_1)" rpy="0 0 ${-pi/4}" connected_to="$(arg arm_id_1)_link8" safety_distance="0.03"/>
+  <xacro:hand arm_id="$(arg arm_id_1)" rpy="0 0 ${-pi/4}" connected_to="$(arg arm_id_1)_link8" safety_distance="0.03"/>
   <!-- left arm with gripper -->
   <xacro:panda_arm arm_id="$(arg arm_id_2)" connected_to="base"  xyz="0 0.5 1" safety_distance="0.03"/>
-  <xacro:hand ns="$(arg arm_id_2)" rpy="0 0 ${-pi/4}" connected_to="$(arg arm_id_2)_link8" safety_distance="0.03"/>
+  <xacro:hand arm_id="$(arg arm_id_2)" rpy="0 0 ${-pi/4}" connected_to="$(arg arm_id_2)_link8" safety_distance="0.03"/>
 </robot>

File: franka_description/robots/hand.urdf.xacro (robot description, xacro)
@@ -2,4 +2,4 @@
 <robot xmlns:xacro="http://www.ros.org/wiki/xacro" name="hand">
   <xacro:include filename="hand.xacro"/>
-  <xacro:hand ns="panda" safety_distance="0.03"/>
+  <xacro:hand arm_id="panda" safety_distance="0.03"/>
 </robot>

File: franka_description/robots/hand.xacro (robot description, xacro)
@@ -2,13 +2,13 @@
 <robot xmlns:xacro="http://www.ros.org/wiki/xacro" name="hand">
   <!-- safety_distance: Minimum safety distance in [m] by which the collision volumes are expanded and which is enforced during robot motions -->
-  <xacro:macro name="hand" params="connected_to:='' ns:='' rpy:='0 0 0' xyz:='0 0 0' safety_distance:=0">
+  <xacro:macro name="hand" params="connected_to:='' arm_id:='panda' rpy:='0 0 0' xyz:='0 0 0' safety_distance:=0">
     <xacro:unless value="${connected_to == ''}">
-      <joint name="${ns}_hand_joint" type="fixed">
+      <joint name="${arm_id}_hand_joint" type="fixed">
         <parent link="${connected_to}"/>
-        <child link="${ns}_hand"/>
+        <child link="${arm_id}_hand"/>
         <origin xyz="${xyz}" rpy="${rpy}"/>
       </joint>
     </xacro:unless>
-    <link name="${ns}_hand">
+    <link name="${arm_id}_hand">
       <visual>
         <geometry>
@@ -53,5 +53,12 @@
       </collision>
     </link>
-    <link name="${ns}_leftfinger">
+    <!-- Define the hand_tcp frame -->
+    <link name="${arm_id}_hand_tcp" />
+    <joint name="${arm_id}_hand_tcp_joint" type="fixed">
+      <origin xyz="0 0 0.1034" rpy="0 0 0" />
+      <parent link="${arm_id}_hand" />
+      <child link="${arm_id}_hand_tcp" />
+    </joint>
+    <link name="${arm_id}_leftfinger">
       <visual>
         <geometry>
@@ -60,5 +67,5 @@
       </visual>
     </link>
-    <link name="${ns}_rightfinger">
+    <link name="${arm_id}_rightfinger">
       <visual>
         <origin xyz="0 0 0" rpy="0 0 ${pi}"/>
@@ -68,18 +75,18 @@
       </visual>
    </link>
-    <joint name="${ns}_finger_joint1" type="prismatic">
-      <parent link="${ns}_hand"/>
-      <child link="${ns}_leftfinger"/>
+    <joint name="${arm_id}_finger_joint1" type="prismatic">
+      <parent link="${arm_id}_hand"/>
+      <child link="${arm_id}_leftfinger"/>
       <origin xyz="0 0 0.0584" rpy="0 0 0"/>
       <axis xyz="0 1 0"/>
-      <limit effort="20" lower="0.0" upper="0.04" velocity="0.2"/>
+      <limit effort="100" lower="0.0" upper="0.04" velocity="0.2"/>
     </joint>
-    <joint name="${ns}_finger_joint2" type="prismatic">
-      <parent link="${ns}_hand"/>
-      <child link="${ns}_rightfinger"/>
+    <joint name="${arm_id}_finger_joint2" type="prismatic">
+      <parent link="${arm_id}_hand"/>
+      <child link="${arm_id}_rightfinger"/>
       <origin xyz="0 0 0.0584" rpy="0 0 0"/>
       <axis xyz="0 -1 0"/>
-      <limit effort="20" lower="0.0" upper="0.04" velocity="0.2"/>
-      <mimic joint="${ns}_finger_joint1" />
+      <limit effort="100" lower="0.0" upper="0.04" velocity="0.2"/>
+      <mimic joint="${arm_id}_finger_joint1" />
     </joint>
   </xacro:macro>

File: franka_description/robots/panda_arm.urdf.xacro (robot description, xacro)
@@ -1,15 +1,17 @@
 <?xml version='1.0' encoding='utf-8'?>
 <robot xmlns:xacro="http://www.ros.org/wiki/xacro" name="panda">
-  <xacro:arg name="arm_id" default="panda" /> <!-- Name of this panda -->
-  <xacro:arg name="hand"   default="false" /> <!-- Should a franka_gripper be mounted at the flange?" -->
-  <xacro:arg name="gazebo" default="false" /> <!-- Is the robot being simulated in gazebo?" -->
-  <xacro:property name="arm_id" value="$(arg arm_id)" />
+  <!-- Name of this panda -->
+  <xacro:arg name="arm_id" default="panda" />
+  <!-- Should a franka_gripper be mounted at the flange?" -->
+  <xacro:arg name="hand" default="false" />
+  <!-- Is the robot being simulated in gazebo?" -->
+  <xacro:arg name="gazebo" default="false" />
   <xacro:unless value="$(arg gazebo)">
     <!-- Create a URDF for a real hardware -->
     <xacro:include filename="$(find franka_description)/robots/panda_arm.xacro" />
-    <xacro:panda_arm arm_id="${arm_id}" safety_distance="0.03"/>
+    <xacro:panda_arm arm_id="$(arg arm_id)" safety_distance="0.03"/>
     <xacro:if value="$(arg hand)">
       <xacro:include filename="$(find franka_description)/robots/hand.xacro"/>
-      <xacro:hand ns="${arm_id}" rpy="0 0 ${-pi/4}" connected_to="${arm_id}_link8" safety_distance="0.03"/>
+      <xacro:hand arm_id="$(arg arm_id)" rpy="0 0 ${-pi/4}" connected_to="$(arg arm_id)_link8" safety_distance="0.03"/>
     </xacro:if>
   </xacro:unless>
@@ -20,9 +22,9 @@
     <xacro:include filename="$(find franka_description)/robots/utils.xacro" />
     <xacro:include filename="$(find franka_description)/robots/panda_gazebo.xacro" />
-    <xacro:panda_arm arm_id="${arm_id}" />
+    <xacro:panda_arm arm_id="$(arg arm_id)" />
     <xacro:if value="$(arg hand)">
-      <xacro:hand ns="${arm_id}" rpy="0 0 ${-pi/4}" connected_to="${arm_id}_link8" />
-      <xacro:gazebo-joint joint="${arm_id}_finger_joint1" transmission="hardware_interface/EffortJointInterface" />
-      <xacro:gazebo-joint joint="${arm_id}_finger_joint2" transmission="hardware_interface/EffortJointInterface" />
+      <xacro:hand arm_id="$(arg arm_id)" rpy="0 0 ${-pi/4}" connected_to="$(arg arm_id)_link8" />
+      <xacro:gazebo-joint joint="$(arg arm_id)_finger_joint1" transmission="hardware_interface/EffortJointInterface" />
+      <xacro:gazebo-joint joint="$(arg arm_id)_finger_joint2" transmission="hardware_interface/EffortJointInterface" />
     </xacro:if>
     <!-- Gazebo requires a joint to a link called "world" for statically mounted robots -->
@@ -31,21 +33,20 @@
       <origin xyz="$(arg xyz)" rpy="$(arg rpy)" />
       <parent link="world" />
-      <child  link="${arm_id}_link0" />
+      <child  link="$(arg arm_id)_link0" />
     </joint>
-    <xacro:gazebo-joint joint="${arm_id}_joint1" transmission="hardware_interface/EffortJointInterface" />
-    <xacro:gazebo-joint joint="${arm_id}_joint2" transmission="hardware_interface/EffortJointInterface" />
-    <xacro:gazebo-joint joint="${arm_id}_joint3" transmission="hardware_interface/EffortJointInterface" />
-    <xacro:gazebo-joint joint="${arm_id}_joint4" transmission="hardware_interface/EffortJointInterface" />
-    <xacro:gazebo-joint joint="${arm_id}_joint5" transmission="hardware_interface/EffortJointInterface" />
-    <xacro:gazebo-joint joint="${arm_id}_joint6" transmission="hardware_interface/EffortJointInterface" />
-    <xacro:gazebo-joint joint="${arm_id}_joint7" transmission="hardware_interface/EffortJointInterface" />
-    <xacro:transmission-franka-state arm_id="${arm_id}" />
-    <xacro:transmission-franka-model arm_id="${arm_id}"
-       root="${arm_id}_joint1"
-       tip="${arm_id}_joint8"
+    <xacro:gazebo-joint joint="$(arg arm_id)_joint1" transmission="hardware_interface/EffortJointInterface" />
+    <xacro:gazebo-joint joint="$(arg arm_id)_joint2" transmission="hardware_interface/EffortJointInterface" />
+    <xacro:gazebo-joint joint="$(arg arm_id)_joint3" transmission="hardware_interface/EffortJointInterface" />
+    <xacro:gazebo-joint joint="$(arg arm_id)_joint4" transmission="hardware_interface/EffortJointInterface" />
+    <xacro:gazebo-joint joint="$(arg arm_id)_joint5" transmission="hardware_interface/EffortJointInterface" />
+    <xacro:gazebo-joint joint="$(arg arm_id)_joint6" transmission="hardware_interface/EffortJointInterface" />
+    <xacro:gazebo-joint joint="$(arg arm_id)_joint7" transmission="hardware_interface/EffortJointInterface" />
+    <xacro:transmission-franka-state arm_id="$(arg arm_id)" />
+    <xacro:transmission-franka-model arm_id="$(arg arm_id)"
+       root="$(arg arm_id)_joint1"
+       tip="$(arg arm_id)_joint8"
      />
     <gazebo>
       <plugin name="gazebo_ros_control" filename="libgazebo_ros_control.so">
-        <robotNamespace>${arm_id}</robotNamespace>
         <controlPeriod>0.001</controlPeriod>
         <robotSimType>franka_gazebo/FrankaHWSim</robotSimType>

File: franka_description/robots/panda_gazebo.xacro (robot description, xacro)
@@ -8,7 +8,14 @@
   <!-- || Penalty-Based Optimization                                || -->
   <!-- || by: Claudio Gaz, Marco Cognetti, Alexander Oliva,         || -->
-  <!-- || Paolo Robuffo Giordano, Alessandro de Lucaa               || -->
+  <!-- || Paolo Robuffo Giordano, Alessandro de Luca                || -->
   <!-- =============================================================== -->
-  <xacro:macro name="panda_arm" params="arm_id:='panda'">
+  <xacro:macro name="panda_arm" params="arm_id:='panda' connected_to:='' xyz:='0 0 0' rpy:='0 0 0'">
+    <xacro:unless value="${not connected_to}">
+      <joint name="${arm_id}_joint_${connected_to}" type="fixed">
+        <parent link="${connected_to}"/>
+        <child link="${arm_id}_link0"/>
+        <origin rpy="${rpy}" xyz="${xyz}"/>
+      </joint>
+    </xacro:unless>
     <link name="${arm_id}_link0">
       <visual>
@@ -251,14 +258,14 @@
     </joint>
   </xacro:macro>
-  <xacro:macro name="hand" params="connected_to:='' ns:='' xyz:='0 0 0' rpy:='0 0 0'">
+  <xacro:macro name="hand" params="connected_to:='' arm_id:='' xyz:='0 0 0' rpy:='0 0 0'">
     <xacro:include filename="$(find franka_description)/robots/utils.xacro"/>
     <xacro:unless value="${connected_to == ''}">
-      <joint name="${ns}_hand_joint" type="fixed">
+      <joint name="${arm_id}_hand_joint" type="fixed">
         <parent link="${connected_to}"/>
-        <child link="${ns}_hand"/>
+        <child link="${arm_id}_hand"/>
         <origin xyz="${xyz}" rpy="${rpy}"/>
       </joint>
     </xacro:unless>
-    <link name="${ns}_hand">
+    <link name="${arm_id}_hand">
       <visual>
         <geometry>
@@ -267,7 +274,6 @@
       </visual>
       <collision>
-        <origin xyz="0.0 0 0.0375" rpy="0 ${pi/2} ${pi/2}"/>
-        <geometry>
-          <box size="0.055 0.04 0.198"  />
+        <geometry>
+          <mesh filename="package://franka_description/meshes/collision/hand.stl" />
         </geometry>
       </collision>
@@ -280,5 +286,35 @@
       </inertial>
     </link>
-    <link name="${ns}_leftfinger">
+    <xacro:macro name="finger-collision" params="sign">
+      <!-- screw mount -->
+      <collision>
+        <origin xyz="0 ${sign}18.5e-3 11e-3" rpy="0 0 0"/>
+        <geometry>
+          <box size="22e-3 15e-3 20e-3" />
+        </geometry>
+      </collision>
+      <!-- cartriage sledge -->
+      <collision>
+        <origin xyz="0 ${sign}6.8e-3 2.2e-3" rpy="0 0 0"/>
+        <geometry>
+          <box size="22e-3 8.8e-3 3.8e-3" />
+        </geometry>
+      </collision>
+      <!-- diagonal finger -->
+      <collision>
+        <origin xyz="0 ${sign}15.9e-3 28.35e-3" rpy="${sign}${pi/6} 0 0"/>
+        <geometry>
+          <box size="17.5e-3 7e-3 23.5e-3" />
+        </geometry>
+      </collision>
+      <!-- rubber tip with which to grasp -->
+      <collision>
+        <origin xyz="0 ${sign}7.58e-3 45.25e-3" rpy="0 0 0"/>
+        <geometry>
+          <box size="17.5e-3 15.2e-3 18.5e-3" />
+        </geometry>
+      </collision>
+    </xacro:macro>
+    <link name="${arm_id}_leftfinger">
       <xacro:inertia-cylinder mass="15e-3" radius="0.01" h="0.04"/>
       <visual>
@@ -287,18 +323,7 @@
         </geometry>
       </visual>
-      <collision>
-        <origin xyz="0 0.015 0.03" rpy="0 0 0"/>
-        <geometry>
-          <box size="0.03 0.005 0.047" />
-        </geometry>
-      </collision>
-      <collision>
-        <origin xyz="0 0.007 0.045" rpy="0 0 0"/>
-        <geometry>
-          <box size="0.03 0.015 0.017" />
-        </geometry>
-      </collision>
-    </link>
-    <link name="${ns}_rightfinger">
+      <xacro:finger-collision sign="+" />
+    </link>
+    <link name="${arm_id}_rightfinger">
       <xacro:inertia-cylinder mass="15e-3" radius="0.01" h="0.04"/>
       <visual>
@@ -308,36 +333,26 @@
         </geometry>
       </visual>
-      <collision>
-        <origin xyz="0 -0.015 0.03" rpy="0 0 0"/>
-        <geometry>
-          <box size="0.03 0.005 0.047" />
-        </geometry>
-      </collision>
-      <collision>
-        <origin xyz="0 -0.007 0.045" rpy="0 0 0"/>
-        <geometry>
-          <box size="0.03 0.015 0.017" />
-        </geometry>
-      </collision>
+      <xacro:finger-collision sign="-" />
     </link>
     <!-- Friction specific material for Rubber/Rubber contact -->
     <!-- See: -->
-    <xacro:gazebo-friction link="${ns}_leftfinger" mu="1.13" />
-    <xacro:gazebo-friction link="${ns}_rightfinger" mu="1.13" />
-    <joint name="${ns}_finger_joint1" type="prismatic">
-      <parent link="${ns}_hand"/>
-      <child link="${ns}_leftfinger"/>
+    <xacro:gazebo-friction link="${arm_id}_leftfinger" mu="1.13" />
+    <xacro:gazebo-friction link="${arm_id}_rightfinger" mu="1.13" />
+    <joint name="${arm_id}_finger_joint1" type="prismatic">
+      <parent link="${arm_id}_hand"/>
+      <child link="${arm_id}_leftfinger"/>
       <origin xyz="0 0 0.0584" rpy="0 0 0"/>
       <axis xyz="0 1 0"/>
-      <limit effort="20" lower="0.0" upper="0.04" velocity="0.2"/>
-      <dynamics damping="0.3"/>
-    </joint>
-    <joint name="${ns}_finger_joint2" type="prismatic">
-      <parent link="${ns}_hand"/>
-      <child link="${ns}_rightfinger"/>
+      <limit effort="100" lower="0.0" upper="0.04" velocity="0.2"/>
+      <dynamics friction="0.0" damping="0.03"/>
+    </joint>
+    <joint name="${arm_id}_finger_joint2" type="prismatic">
+      <parent link="${arm_id}_hand"/>
+      <child link="${arm_id}_rightfinger"/>
       <origin xyz="0 0 0.0584" rpy="0 0 0"/>
       <axis xyz="0 -1 0"/>
-      <limit effort="20" lower="0.0" upper="0.04" velocity="0.2"/>
-      <dynamics damping="0.3"/>
+      <limit effort="100" lower="0.0" upper="0.04" velocity="0.2"/>
+      <dynamics friction="0.0" damping="0.03"/>
+      <mimic joint="${arm_id}_finger_joint1" />
     </joint>
   </xacro:macro>

File: franka_description/robots/utils.xacro (robot description, xacro)
@@ -33,5 +33,5 @@
               <!-- penetration depth to keep the grasping stable -->
               <max_vel>0</max_vel>
-              <min_depth>0.003</min_depth>
+              <min_depth>0.001</min_depth>
             </ode>
           </contact>
